File: hw/kicad/v5.0/hv.kicad_sch (KiCad schematic)
At the start: 17 parts, among them P2 CONN_01X02, Q5 IRLML6344, U3 SI8621

Commit message: update gerber files
Other:
- note removed: "Negare itirp via software!!!"
Changed lines of the file:
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@@
-		)
-	)
-	(text "Negare itirp via software!!!"
-		(exclude_from_sim no)
-		(at 172.72 85.09 0)
-		(effects
-			(font
-				(size 1.27 1.27)
-			)
-			(justify left bottom)
 		)
 	)
