File: hw/kicad/v5.0/stmbl_4.0.kicad_sch (KiCad schematic)
At the start: 2 parts, among them U234 fan, U33 heatsink

Commit message: update gerber files
Parts:
- U234: Voltage 12V -> 124V
Changed lines of the file:
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@@
 		)
 		(property "Footprint" "stmbl:radial fan"
-			(at 142.24 99.06 0)
+			(at 143.764 106.426 0)
 			(effects
 				(font
@@
 			)
 		)
-		(property "Voltage" "12V"
+		(property "Voltage" "124V"
 			(at 142.24 99.06 0)
 			(effects
