File: hw/kicad/v5.0/supply.kicad_sch (KiCad schematic)
At the start: 65 parts, among them P3 CONN_01X02, U13 RT8259, U2 zldo1117, U24 RT8259, U28 RT8259

Commit message: update gerber files
Parts:
- R155, R156, R157, R158: now not fitted; now left out of the parts list
Changed lines of the file:
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@@
 					(size 1.27 1.27)
 				)
+				(hide yes)
 			)
 		)
@@
 		(unit 1)
 		(exclude_from_sim no)
-		(in_bom yes)
+		(in_bom no)
 		(on_board yes)
-		(dnp no)
+		(dnp yes)
 		(property "Reference" "R158"
 			(at 135.89 49.53 90)
@@
 		(unit 1)
 		(exclude_from_sim no)
-		(in_bom yes)
+		(in_bom no)
 		(on_board yes)
-		(dnp no)
+		(dnp yes)
 		(property "Reference" "R155"
 			(at 120.65 49.53 90)
@@
 			)
 		)
-		(property "Description" ""
+		(property "Description" "NM"
 			(at 16.51 127 0)
 			(effects
@@
 		(unit 1)
 		(exclude_from_sim no)
-		(in_bom yes)
+		(in_bom no)
 		(on_board yes)
-		(dnp no)
+		(dnp yes)
 		(property "Reference" "R156"
 			(at 125.73 49.53 90)
@@
 		(unit 1)
 		(exclude_from_sim no)
-		(in_bom yes)
+		(in_bom no)
 		(on_board yes)
-		(dnp no)
+		(dnp yes)
 		(property "Reference" "R157"
 			(at 130.81 49.53 90)
