File: hw/kicad/v5.0/f3.kicad_sch (KiCad schematic)
At the start: 35 parts, among them P11 USB_C_Receptacle_USB2.0, P12 CONN_01X04, P7 CONN_01X04, T1 testpoint, T2 testpoint, T44 testpoint, T45 testpoint, T46 testpoint, U21 USBLC6-4SC6, U25 STM32F303CBTx, U29 USBLC6-4SC6, Y1 8M

Commit message: 4 pin connectors on f3 side changed to smd
Parts:
- P12, P7: footprint stmbl:Pin_Header_Straight_1x04 -> stmbl:Pin_Header_Straight_1x04_smd
Changed lines of the file:
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@@
 			)
 		)
-		(property "Footprint" "stmbl:Pin_Header_Straight_1x04"
+		(property "Footprint" "stmbl:Pin_Header_Straight_1x04_smd"
 			(at 137.16 134.62 0)
 			(effects
@@
 			)
 		)
-		(property "Footprint" "stmbl:Pin_Header_Straight_1x04"
+		(property "Footprint" "stmbl:Pin_Header_Straight_1x04_smd"
 			(at 270.51 105.41 0)
 			(effects

Commit message: check important points of drc
Parts:
- P7: now left out of the parts list
Changed lines of the file:
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@@
 		(unit 1)
 		(exclude_from_sim no)
-		(in_bom yes)
+		(in_bom no)
 		(on_board yes)
 		(dnp no)
